Commit message: cobot updated

File: cobot_simulation/urdf/cobot.urdf (robot description, URDF)
Before this commit: robot cobot, 5 links, 4 joints
Links:
- removed link base_link
- removed link link1
- removed link link2
- removed link link3
- removed link link4
- added link world
Joints:
- removed joint base_link__link1
- removed joint link1__link2
- removed joint link2__link3
- removed joint link3__link4
- added joint fixed: type fixed, parent world, child base_link
